File: pcb/dcc_sniffer_nano.brd (EAGLE design)
At the start: 19.1 x 53.3 mm, 8 parts, among them X1 RT034 Typ 086

Commit message: bugfix: assign to IRQ input pin
Connections:
- net N$3: now also ARDUINO1.11; no longer ARDUINO1.8
Routing:
- net N$3: track 16.3 -> 28.0 mm
- net +5V: track 41.5 -> 40.6 mm
Other:
- board text added: "+"
- board text added: "DCC Sniffer 115200 Bps"
- board text added: "OMC Adorf 2021 Rev 1.0"
- board text removed: "DCC Sniffer Nano"
Changed lines of the file:
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@@
 <wire x1="19.05" y1="53.34" x2="0" y2="53.34" width="0" layer="20"/>
 <wire x1="0" y1="53.34" x2="0" y2="0" width="0" layer="20"/>
-<text x="16.51" y="45.72" size="1.778" layer="21" font="vector" ratio="15" rot="R90">track</text>
-<text x="5.08" y="5.08" size="1.778" layer="21" font="vector" ratio="15">DCC
-Sniffer
-Nano</text>
+<text x="17.145" y="46.355" size="1.27" layer="21" font="vector" ratio="15" rot="R90">track</text>
+<text x="4.445" y="6.985" size="1.4224" layer="21" font="vector" ratio="15">OMC Adorf
+2021
+Rev 1.0</text>
+<text x="15.24" y="16.51" size="1.6764" layer="26" font="vector" ratio="12" rot="MR270">DCC Sniffer
+115200 Bps</text>
+<text x="13.97" y="49.53" size="2.1844" layer="21" font="vector" ratio="15">+</text>
 </plain>
 <attributes>
@@
 <attribute name="OC_FARNELL" value="1328376" x="9.525" y="20.955" size="1.778" layer="27" rot="R90" display="off"/>
 <attribute name="MPN" value="6N137" x="9.525" y="20.955" size="1.778" layer="27" rot="R90" display="off"/>
-<attribute name="NAME" x="12.446" y="15.621" size="1.27" layer="25" ratio="10" rot="R180"/>
+<attribute name="NAME" x="13.081" y="15.621" size="1.27" layer="25" ratio="10" rot="R180"/>
 </element>
 <element name="R1" library="resistor" package="0207/10" value="1k" x="13.335" y="38.1" smashed="yes" rot="R270">
@@
 <attribute name="VENDOR#" value="Metz Connect#31086102" x="11.43" y="48.895" size="1.778" layer="27" rot="R180" display="off"/>
 <attribute name="DIST#DIGIKEY#" value="" x="11.43" y="48.895" size="1.778" layer="27" rot="R180" display="off"/>
-<attribute name="NAME" x="5.715" y="52.308125" size="1.27" layer="25" font="vector" rot="R180"/>
+<attribute name="NAME" x="5.715" y="51.673125" size="1.27" layer="25" font="vector" rot="R180"/>
 </element>
 <element name="C1" library="resistor" package="C025-025X050" value="1n" x="12.7" y="27.94" smashed="yes">
@@
 <vertex x="19.05" y="53.34"/>
 </polygon>
+<via x="1.27" y="52.07" extent="1-16" drill="0.6" diameter="0.8128" shape="octagon"/>
+<via x="17.78" y="52.07" extent="1-16" drill="0.6" diameter="0.8128" shape="octagon"/>
+<via x="1.27" y="1.27" extent="1-16" drill="0.6" diameter="0.8128" shape="octagon"/>
+<via x="17.78" y="1.27" extent="1-16" drill="0.6" diameter="0.8128" shape="octagon"/>
+<via x="8.89" y="15.24" extent="1-16" drill="0.6" diameter="0.8128" shape="octagon"/>
 </signal>
 <signal name="+5V">
@@
 <wire x1="13.335" y1="30.48" x2="8.255" y2="30.48" width="0.8128" layer="1"/>
 <wire x1="8.255" y1="30.48" x2="8.255" y2="27.94" width="0.8128" layer="1"/>
-<wire x1="8.255" y1="27.94" x2="9.525" y2="26.67" width="0.4064" layer="1"/>
-<via x="9.525" y="17.145" extent="1-16" drill="0.6" shape="octagon"/>
+<via x="8.89" y="17.145" extent="1-16" drill="0.6" shape="octagon"/>
 <wire x1="7.62" y1="27.94" x2="8.255" y2="27.94" width="0.4064" layer="1"/>
-<wire x1="5.715" y1="17.145" x2="9.525" y2="17.145" width="0.4064" layer="16"/>
-<wire x1="9.525" y1="17.145" x2="9.525" y2="26.67" width="0.4064" layer="1"/>
+<wire x1="5.715" y1="17.145" x2="8.89" y2="17.145" width="0.4064" layer="16"/>
+<wire x1="8.255" y1="27.94" x2="8.89" y2="27.305" width="0.8128" layer="1"/>
+<wire x1="8.89" y1="27.305" x2="8.89" y2="17.145" width="0.8128" layer="1"/>
 </signal>
 <signal name="N$1">
@@
 <contactref element="OK1" pad="6"/>
 <contactref element="R2" pad="1"/>
-<contactref element="ARDUINO1" pad="8"/>
-<wire x1="1.905" y1="22.225" x2="5.715" y2="22.225" width="0.4064" layer="16"/>
 <wire x1="5.715" y1="22.225" x2="6.35" y2="22.225" width="0.4064" layer="16"/>
 <wire x1="6.35" y1="33.02" x2="6.35" y2="26.67" width="0.4064" layer="16"/>
-<wire x1="7.62" y1="23.495" x2="6.35" y2="22.225" width="0.4064" layer="16"/>
 <wire x1="6.35" y1="26.67" x2="7.62" y2="25.4" width="0.4064" layer="16"/>
-<wire x1="7.62" y1="25.4" x2="7.62" y2="23.495" width="0.4064" layer="16"/>
+<wire x1="7.62" y1="25.4" x2="7.62" y2="22.86" width="0.4064" layer="16"/>
+<contactref element="ARDUINO1" pad="11"/>
+<wire x1="1.905" y1="14.605" x2="6.985" y2="14.605" width="0.4064" layer="1"/>
+<wire x1="6.985" y1="14.605" x2="7.62" y2="15.24" width="0.4064" layer="1"/>
+<wire x1="7.62" y1="15.24" x2="7.62" y2="21.59" width="0.4064" layer="1"/>
+<wire x1="7.62" y1="21.59" x2="6.985" y2="22.225" width="0.4064" layer="1"/>
+<wire x1="6.985" y1="22.225" x2="5.715" y2="22.225" width="0.4064" layer="1"/>
+<wire x1="7.62" y1="22.86" x2="6.985" y2="22.225" width="0.4064" layer="16"/>
+<wire x1="6.985" y1="22.225" x2="5.715" y2="22.225" width="0.4064" layer="16"/>
 </signal>
 <signal name="N$4">
